File: pcb/power_xt60_frontpanel.sch (EAGLE design)
At the start: 21 parts, among them X1 SOLDERPAD4X5, X10 SOLDERPAD4X5, X11 SOLDERPAD4X5, X12 SOLDERPAD4X5, X2 SOLDERPAD4X5, X3 SOLDERPAD4X5, X4 SOLDERPAD4X5, X5 SOLDERPAD4X5, X6 SOLDERPAD4X5, X7 SOLDERPAD4X5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

Commit message: Revison 2
Connections:
- net GND: now also H1.-, H2.-, H3.-, H4.-, H5.-
- net VCC: now also H1.+, H2.+, H3.+, H4.+, H5.+
Changed lines of the file:
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@@
 <part name="X11" library="M2M-Connectors" deviceset="SOLDERPAD" device="4X5"/>
 <part name="X12" library="M2M-Connectors" deviceset="SOLDERPAD" device="4X5"/>
+<part name="GND2" library="M2M-Power" deviceset="GND" device=""/>
+<part name="SUPPLY2" library="M2M-Power" deviceset="VCC" device=""/>
 </parts>
 <sheets>
@@
 <attribute name="SHEET" x="230.505" y="5.08" size="2.54" layer="94"/>
 </instance>
-<instance part="H1" gate="G$1" x="134.62" y="116.84" smashed="yes">
-<attribute name="NAME" x="132.08" y="122.682" size="1.778" layer="95"/>
-<attribute name="VALUE" x="132.08" y="109.22" size="1.778" layer="96"/>
-</instance>
-<instance part="H2" gate="G$1" x="134.62" y="99.06" smashed="yes">
-<attribute name="NAME" x="132.08" y="104.902" size="1.778" layer="95"/>
-<attribute name="VALUE" x="132.08" y="91.44" size="1.778" layer="96"/>
-</instance>
-<instance part="H3" gate="G$1" x="134.62" y="81.28" smashed="yes">
-<attribute name="NAME" x="132.08" y="87.122" size="1.778" layer="95"/>
-<attribute name="VALUE" x="132.08" y="73.66" size="1.778" layer="96"/>
-</instance>
-<instance part="H4" gate="G$1" x="134.62" y="63.5" smashed="yes">
-<attribute name="NAME" x="132.08" y="69.342" size="1.778" layer="95"/>
-<attribute name="VALUE" x="132.08" y="55.88" size="1.778" layer="96"/>
-</instance>
-<instance part="H5" gate="G$1" x="134.62" y="134.62" smashed="yes">
-<attribute name="NAME" x="132.08" y="140.462" size="1.778" layer="95"/>
-<attribute name="VALUE" x="132.08" y="127" size="1.778" layer="96"/>
+<instance part="H1" gate="G$1" x="144.78" y="116.84" smashed="yes">
+<attribute name="NAME" x="142.24" y="122.682" size="1.778" layer="95"/>
+<attribute name="VALUE" x="142.24" y="109.22" size="1.778" layer="96"/>
+</instance>
+<instance part="H2" gate="G$1" x="144.78" y="99.06" smashed="yes">
+<attribute name="NAME" x="142.24" y="104.902" size="1.778" layer="95"/>
+<attribute name="VALUE" x="142.24" y="91.44" size="1.778" layer="96"/>
+</instance>
+<instance part="H3" gate="G$1" x="144.78" y="81.28" smashed="yes">
+<attribute name="NAME" x="142.24" y="87.122" size="1.778" layer="95"/>
+<attribute name="VALUE" x="142.24" y="73.66" size="1.778" layer="96"/>
+</instance>
+<instance part="H4" gate="G$1" x="144.78" y="63.5" smashed="yes">
+<attribute name="NAME" x="142.24" y="69.342" size="1.778" layer="95"/>
+<attribute name="VALUE" x="142.24" y="55.88" size="1.778" layer="96"/>
+</instance>
+<instance part="H5" gate="G$1" x="144.78" y="134.62" smashed="yes">
+<attribute name="NAME" x="142.24" y="140.462" size="1.778" layer="95"/>
+<attribute name="VALUE" x="142.24" y="127" size="1.778" layer="96"/>
 </instance>
 <instance part="SUPPLY1" gate="G$1" x="63.5" y="142.24" smashed="yes">
@@
 <attribute name="VALUE" x="101.6" y="68.58" size="1.778" layer="96"/>
 <attribute name="NAME" x="101.6" y="76.962" size="1.778" layer="95"/>
+</instance>
+<instance part="GND2" gate="1" x="134.62" y="48.26" smashed="yes">
+<attribute name="VALUE" x="134.62" y="48.006" size="1.778" layer="96" align="top-center"/>
+</instance>
+<instance part="SUPPLY2" gate="G$1" x="132.08" y="139.7" smashed="yes">
+<attribute name="VALUE" x="132.08" y="142.494" size="1.778" layer="96" align="bottom-center"/>
 </instance>
 </instances>
@@
 <junction x="63.5" y="63.5"/>
 </segment>
+<segment>
+<pinref part="H5" gate="G$1" pin="+"/>
+<wire x1="137.16" y1="137.16" x2="132.08" y2="137.16" width="0.1524" layer="91"/>
+<wire x1="132.08" y1="137.16" x2="132.08" y2="119.38" width="0.1524" layer="91"/>
+<pinref part="H4" gate="G$1" pin="+"/>
+<wire x1="132.08" y1="119.38" x2="132.08" y2="101.6" width="0.1524" layer="91"/>
+<wire x1="132.08" y1="101.6" x2="132.08" y2="83.82" width="0.1524" layer="91"/>
+<wire x1="132.08" y1="83.82" x2="132.08" y2="66.04" width="0.1524" layer="91"/>
+<wire x1="132.08" y1="66.04" x2="137.16" y2="66.04" width="0.1524" layer="91"/>
+<pinref part="H3" gate="G$1" pin="+"/>
+<wire x1="137.16" y1="83.82" x2="132.08" y2="83.82" width="0.1524" layer="91"/>
+<junction x="132.08" y="83.82"/>
+<pinref part="H2" gate="G$1" pin="+"/>
+<wire x1="137.16" y1="101.6" x2="132.08" y2="101.6" width="0.1524" layer="91"/>
+<junction x="132.08" y="101.6"/>
+<pinref part="H1" gate="G$1" pin="+"/>
+<wire x1="137.16" y1="119.38" x2="132.08" y2="119.38" width="0.1524" layer="91"/>
+<junction x="132.08" y="119.38"/>
+<pinref part="SUPPLY2" gate="G$1" pin="VCC"/>
+<wire x1="132.08" y1="139.7" x2="132.08" y2="137.16" width="0.1524" layer="91"/>
+<junction x="132.08" y="137.16"/>
+</segment>
 </net>
 <net name="GND" class="0">
@@
 <junction x="96.52" y="63.5"/>
 </segment>
+<segment>
+<pinref part="H5" gate="G$1" pin="-"/>
+<wire x1="137.16" y1="132.08" x2="134.62" y2="132.08" width="0.1524" layer="91"/>
+<pinref part="H4" gate="G$1" pin="-"/>
+<wire x1="134.62" y1="132.08" x2="134.62" y2="114.3" width="0.1524" layer="91"/>
+<wire x1="134.62" y1="114.3" x2="134.62" y2="96.52" width="0.1524" layer="91"/>
+<wire x1="134.62" y1="96.52" x2="134.62" y2="78.74" width="0.1524" layer="91"/>
+<wire x1="134.62" y1="78.74" x2="134.62" y2="60.96" width="0.1524" layer="91"/>
+<wire x1="134.62" y1="60.96" x2="137.16" y2="60.96" width="0.1524" layer="91"/>
+<pinref part="H3" gate="G$1" pin="-"/>
+<wire x1="137.16" y1="78.74" x2="134.62" y2="78.74" width="0.1524" layer="91"/>
+<junction x="134.62" y="78.74"/>
+<pinref part="H2" gate="G$1" pin="-"/>
+<wire x1="137.16" y1="96.52" x2="134.62" y2="96.52" width="0.1524" layer="91"/>
+<junction x="134.62" y="96.52"/>
+<pinref part="H1" gate="G$1" pin="-"/>
+<wire x1="137.16" y1="114.3" x2="134.62" y2="114.3" width="0.1524" layer="91"/>
+<junction x="134.62" y="114.3"/>
+<pinref part="GND2" gate="1" pin="GND"/>
+<wire x1="134.62" y1="60.96" x2="134.62" y2="50.8" width="0.1524" layer="91"/>
+<junction x="134.62" y="60.96"/>
+</segment>
 </net>
